File: GAME.brd (EAGLE design)
At the start: 138 x 54 mm, 33 parts, among them J1 Digital_0_7, J2 Analog, J3 Digital_8_13, J4 Power, J5 ICSP, J6 M05X2PTH

Commit message: Fixed OLED pinout for v1.1 release
Parts:
- moved J6 1.27 mm to (61.1, 41.9)
Connections:
- net 5V: now also J6.2; no longer J6.1
- net D2: now also J6.10; no longer J6.9
- net D3: now also J6.9; no longer J6.10
- net D4: now also J6.4; no longer J6.3
- net D5: now also J6.3; no longer J6.4
- net D7: now also J6.7; no longer J6.8
- net GND: now also J6.1; no longer J6.2
- net MISO: now also J6.6; no longer J6.5
- net MOSI: now also J6.5; no longer J6.6
- net SCK: now also J6.8; no longer J6.7
Routing:
- net SCK: track 41.5 -> 50.8 mm, vias 1 -> 0
- net MOSI: track 47.6 -> 42.6 mm, vias 1 -> 0
- net MISO: track 38.9 -> 43.3 mm, vias 1 -> 0
- net D4: track 34.2 -> 30.3 mm
- net D2: track 29.6 -> 26.0 mm, vias 0 -> 1
- net 5V: track 133.1 -> 135.3 mm
- net D5: track 28.5 -> 27.2 mm
- net D7: track 17.6 -> 16.9 mm
Other:
- board text added: "v1.1"
- board text removed: "v1.0"
